File: esp32controller.sch (KiCad schematic (older format))
At the start: 115 parts, among them J1 Conn_01x06, J10 Conn_01x06_Female, J11 Conn_01x04, J12 Conn_01x04, J13 Conn_01x04, J14 Conn_01x04, J15 Conn_01x04, J16 Conn_02x03_Odd_Even, J17 Conn_02x03_Odd_Even, J18 Conn_02x03_Odd_Even, J19 Conn_02x03_Odd_Even, J2 USB_B, J20 Conn_02x03_Odd_Even, J3 Conn_01x03, J4 Conn_01x03, J5 Conn_01x03, J6 Conn_02x16_Odd_Even, J7 Conn_01x04_Female, J8 Conn_01x32, J9 Micro_SD_Card_Det, Q1 Q_NPN_BEC, Q2 Q_NPN_BEC, Q3 Q_NMOS_GDS, Q4 Q_NMOS_GDS, Q5 Q_NMOS_GDS, SW1 SW_Push, U1 CH340C, U2 ESP32-WROOM, U3 74HC595, U4 74HC595, U5 74HC595, U6 74HC595, U7 TPS560430, U8 TLV1117-33

Commit message: Shuffled pins, added Display Connector and more FETs, Supplied Shiftregister with 5V for higher Gate Drive voltage
Parts:
- removed J6: Conn_02x16_Odd_Even, Connector_PinHeader_2.54mm:PinHeader_2x16_P2.54mm_Vertical, symbol Connector_Generic:Conn_02x16_Odd_Even
- removed Q1, Q2: Q_NPN_BEC, Package_TO_SOT_SMD:SOT-23, symbol Device:Q_NPN_BEC
- added J21: EXP1, Connector_PinHeader_2.54mm:PinHeader_2x05_P2.54mm_Vertical, symbol Connector_Generic:Conn_02x05_Odd_Even
- added J22: EXP2, Connector_PinHeader_2.54mm:PinHeader_2x05_P2.54mm_Vertical, symbol Connector_Generic:Conn_02x05_Odd_Even
- added J23: E0_FAN, Connector_PinHeader_2.54mm:PinHeader_1x02_P2.54mm_Vertical, symbol Connector:Conn_01x02_Male
- added J24: E1_FAN, Connector_PinHeader_2.54mm:PinHeader_1x02_P2.54mm_Vertical, symbol Connector:Conn_01x02_Male
- added J25: Controller_FAN, Connector_PinHeader_2.54mm:PinHeader_1x02_P2.54mm_Vertical, symbol Connector:Conn_01x02_Male
- added J6: con, Connector_PinHeader_2.54mm:PinHeader_2x05_P2.54mm_Vertical, symbol Connector_Generic:Conn_02x05_Odd_Even
- added Q1, Q2: BC817, Package_TO_SOT_SMD:SOT-23, symbol Transistor_BJT:BC817
- added Q6, Q7, Q8: SI2300, Package_TO_SOT_SMD:SOT-23, symbol Device:Q_NMOS_GSD
- added R37, R39, R41: 10, Resistor_SMD:R_0805_2012Metric, symbol Device:R
- added R38, R40, R42: 100k, Resistor_SMD:R_0805_2012Metric, symbol Device:R
- added R43, R44: 2.4k, Resistor_SMD:R_0805_2012Metric, symbol Device:R
- C1, C10, C11, C12, C13, C14, C15, C17, C20, C6, C7, C8, C9: footprint Capacitor_SMD:C_0603_1608Metric -> Capacitor_SMD:C_0805_2012Metric
- R1, R10, R11, R12, R13, R14, R15, R18, R19, R2, R20, R21, R22, R23, R24, R25, R26, R27, R28, R29, R3, R30, R31, R32, R33, R34, R35, R36, R4, R5, R6, R7, R8, R9: footprint Resistor_SMD:R_0603_1608Metric -> Resistor_SMD:R_0805_2012Metric
- R16, R17: footprint Resistor_SMD:R_1206_3216Metric -> Resistor_SMD:R_0805_2012Metric
Connections:
- net labels added: +5VD, BTNE, But1, But2, Buzzer, KILLSW, LCD4, LCD5, LCD6, LCD7, LCDE, LCDRS, SD_DET
- net labels removed: BED, FAN, HEATER, HSPI_MISO, HSPI_MOSI, HSPI_SCK, HSPI_SS
- wire segments 355 -> 364
- no-connect marks 18 -> 19
Other:
- moved on the sheet: C12, C13, C14, C15, C16, D3, D4, MK1, MK2, MK3, MK4, R14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
