File: esp32controller.kicad_pcb (KiCad board)
At the start: 2 copper layers, 101.6 x 82.6 mm, 115 parts, among them J1 Conn_01x06, J10 Conn_01x06_Female, J11 Conn_01x04, J12 Conn_01x04, J13 Conn_01x04, J14 Conn_01x04, J15 Conn_01x04, J16 Conn_02x03_Odd_Even, J17 Conn_02x03_Odd_Even, J18 Conn_02x03_Odd_Even, J19 Conn_02x03_Odd_Even, J2 USB_B, J20 Conn_02x03_Odd_Even, J3 Conn_01x03, J4 Conn_01x03, J5 Conn_01x03, J6 Conn_02x16_Odd_Even, J7 Conn_01x04_Female, J8 Conn_01x32, J9 Micro_SD_Card_Det, Q1 Q_NPN_BEC, Q2 Q_NPN_BEC, Q3 Q_NMOS_GDS, Q4 Q_NMOS_GDS, Q5 Q_NMOS_GDS, SW1 SW_Push, U1 CH340C, U2 ESP32-WROOM, U3 74HC595, U4 74HC595, U5 74HC595, U6 74HC595, U7 TPS560430, U8 TLV1117-33

Commit message: Routed R3 Board
Parts:
- added J21: EXP1, Connector_PinHeader_2.54mm:PinHeader_2x05_P2.54mm_Vertical, F.Cu at (137.2, 83.8)
- added J22: EXP2, Connector_PinHeader_2.54mm:PinHeader_2x05_P2.54mm_Vertical, F.Cu at (109.2, 53.8)
- added J23: E0_FAN, Connector_PinHeader_2.54mm:PinHeader_1x02_P2.54mm_Vertical, F.Cu at (199.4, 80.0)
- added J24: E1_FAN, Connector_PinHeader_2.54mm:PinHeader_1x02_P2.54mm_Vertical, F.Cu at (199.4, 82.5)
- added J25: Controller_FAN, Connector_PinHeader_2.54mm:PinHeader_1x02_P2.54mm_Vertical, F.Cu at (199.4, 85.1)
- added Q6: SI2300, Package_TO_SOT_SMD:SOT-23, F.Cu at (201.6, 98.0)
- added Q7: SI2300, Package_TO_SOT_SMD:SOT-23, F.Cu at (201.6, 94.0)
- added Q8: SI2300, Package_TO_SOT_SMD:SOT-23, F.Cu at (201.6, 90.0)
- added R37: 10, Resistor_SMD:R_0805_2012Metric, F.Cu at (197.5, 97.0)
- added R38: 100k, Resistor_SMD:R_0805_2012Metric, F.Cu at (197.5, 99.0)
- added R39: 10, Resistor_SMD:R_0805_2012Metric, F.Cu at (197.5, 93.0)
- added R40: 100k, Resistor_SMD:R_0805_2012Metric, F.Cu at (197.5, 95.0)
- added R41: 10, Resistor_SMD:R_0805_2012Metric, F.Cu at (197.5, 89.0)
- added R42: 100k, Resistor_SMD:R_0805_2012Metric, F.Cu at (197.5, 91.0)
- added R43: 2.4k, Resistor_SMD:R_0805_2012Metric, F.Cu at (125.6, 59.0)
- added R44: 2.4k, Resistor_SMD:R_0805_2012Metric, F.Cu at (137.6, 59.0)
- C1, C10, C11, C12, C13, C14, C15, C17, C20, C6, C7, C8, C9: footprint Capacitor_SMD:C_0603_1608Metric -> Capacitor_SMD:C_0805_2012Metric
- J6: value Conn_02x16_Odd_Even -> con; footprint Connector_PinHeader_2.54mm:PinHeader_2x16_P2.54mm_Vertical -> Connector_PinHeader_2.54mm:PinHeader_2x05_P2.54mm_Vertical
- Q1, Q2: value Q_NPN_BEC -> BC817
- R1, R10, R11, R12, R13, R14, R15, R18, R19, R2, R20, R21, R22, R23, R24, R25, R26, R27, R28, R29, R3, R30, R31, R32, R33, R34, R35, R36, R4, R5, R6, R7, R8, R9: footprint Resistor_SMD:R_0603_1608Metric -> Resistor_SMD:R_0805_2012Metric
- R16, R17: footprint Resistor_SMD:R_1206_3216Metric -> Resistor_SMD:R_0805_2012Metric
- moved R10 65.2 mm to (127.5, 78.0), turned to 180 degrees
- moved R14 36.7 mm to (127.5, 76.0), turned to 180 degrees
- moved R15 35.2 mm to (127.5, 74.0), turned to 180 degrees
- moved J6 15.5 mm to (142.2, 86.4)
- moved C6 13.7 mm to (141.7, 97.8)
- moved J8 10.2 mm to (154.9, 98.1)
- moved U3 10.0 mm to (163.9, 88.5)
- moved U4 10.0 mm to (172.9, 88.5)
- moved U5 10.0 mm to (182.2, 88.5)
- moved U6 10.0 mm to (190.9, 88.5)
- moved C12 10.0 mm to (159.6, 86.5)
- moved C13 10.0 mm to (168.6, 86.5)
- moved C14 10.0 mm to (186.6, 86.5)
- moved C15 10.0 mm to (177.6, 86.5)
- moved C7 6.28 mm to (195.6, 75.9)
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Connections:
- A1 pad 16: /Q2 -> /Q0
- A1 pad 9: /Q0 -> /Q2
- A2 pad 16: /Q5 -> /Q3
- A2 pad 9: /Q3 -> /Q5
- A3 pad 16: /Q8 -> /Q6
- A3 pad 9: /Q6 -> /Q8
- A4 pad 16: /Q11 -> /Q9
- A4 pad 9: /Q9 -> /Q11
- A5 pad 16: /Q14 -> /Q12
- A5 pad 9: /Q12 -> /Q14
- C14 pad 1: VCC -> +5V
- C15 pad 1: VCC -> +5V
- C19 pad 1: +5V -> +5VD
- C21 pad 1: Net-(C21-Pad1) -> +5V
- J6 pad 1: +24V -> VCC
- J6 pad 10: GND -> /TXD
- J6 pad 3: VCC -> /EN
- J6 pad 4: GND -> (no net)
- J6 pad 5: /EN -> /BCLK
- J6 pad 6: /IO25 -> /IO4
- J6 pad 7: /IO26 -> /IO16
- J6 pad 8: /FAN -> /IO17
- J6 pad 9: VCC -> /RXD
- JP1 pad 1: +5V -> +5VD
- JP1 pad 2: Net-(C21-Pad1) -> +5V
- L1 pad 2: +5V -> +5VD
- R10 pad 2: /HEATER -> /Buzzer
- R14 pad 2: /IO22 -> /But2
- R15 pad 2: /IO21 -> /But1
- R16 pad 1: +24V -> Net-(R16-Pad1)
- R17 pad 1: /+24V2 -> Net-(R17-Pad1)
- R18 pad 2: /FAN -> /Q17
- R19 pad 2: /FAN -> /Q17
- R20 pad 2: /HEATER -> /Q16
- R21 pad 2: /HEATER -> /Q16
- R22 pad 1: +5V -> +5VD
- R23 pad 2: /BED -> /Q18
- R25 pad 2: /BED -> /Q18
- R27 pad 2: /Q0 -> /Q2
- R28 pad 2: /Q3 -> /Q5
- R29 pad 2: /Q6 -> /Q8
- R30 pad 2: /Q9 -> /Q11
- R31 pad 2: /Q12 -> /Q14
- U2 pad 10: /IO25 -> /BTNE
- U2 pad 12: /FAN -> /IO27
- U2 pad 13: /HSPI_SCK -> /IO14
- U2 pad 14: /HSPI_MISO -> /IO12
- U2 pad 16: /HSPI_MOSI -> /IO13
- U2 pad 23: /HSPI_SS -> /IO15
- U2 pad 24: /HEATER -> /Buzzer
- U2 pad 26: /BED -> /IO4
- U2 pad 33: /IO21 -> /But1
- U2 pad 36: /IO22 -> /But2
- U5 pad 10: VCC -> +5V
- U5 pad 16: VCC -> +5V
- U6 pad 10: VCC -> +5V
- U6 pad 16: VCC -> +5V
- U8 pad 3: Net-(C21-Pad1) -> +5V
Routing:
- net /Q18: track 9.21 -> 127.6 mm
- net /Q17: track 6.11 -> 116.5 mm
- net /HEATER: track 108.4 -> 0.00 mm, vias 1 -> 0
- net /BED: track 105.2 -> 0.00 mm, vias 4 -> 0
- net /Q16: track 15.3 -> 109.8 mm
- net /FAN: track 86.7 -> 0.00 mm, vias 3 -> 0
- net /IO22: track 73.7 -> 0.00 mm, vias 2 -> 0
- net /IO21: track 65.1 -> 0.00 mm, vias 2 -> 0
- net /IO4: track 0.00 -> 59.3 mm, vias 0 -> 2
- net /IO23: track 74.9 -> 29.8 mm, vias 2 -> 0
- net /IO18: track 72.3 -> 27.6 mm
- net /IO5: track 61.6 -> 20.4 mm, vias 0 -> 1
- net /But2: track 0.00 -> 40.6 mm
- net /IO19: track 72.6 -> 34.4 mm, vias 3 -> 2
- net /Q6: track 67.3 -> 29.3 mm
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- added copper zone on F.Cu, net +5VD
- removed copper zone on F.Cu, net +5V
